File: hw/IRQF401RCT6v1.011.revB/IRQF401RCT6.brd (EAGLE design)
At the start: 74 x 53 mm, 105 parts, among them IC1 STM32F401RCT, IC2 LM1117IMPX-3.3, IC3 LM1117MPX-5.0, J2 RJ11, J3 RJ11, P1 FSM, Q1 8MHz, Q2 32.768kHz, Q3 BC846BSMD, Q4 BSS84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

Commit message: rev
New revision
Parts:
- removed Q1: 8MHz, crystal:HC49/S
- removed Q2: 32.768kHz, crystal:TC26H
- added Y1: 8MHz, crystal:HC49/S
- added Y2: 32.768kHz, crystal:TC26H
- moved JP5 1.05 mm to (35.2, 45.2)
- moved JP3 0.30 mm to (35.2, 41.5)
- moved R1 0.25 mm to (51.0, 47.4)
- moved R16 0.25 mm to (37.4, 48.1)
Connections:
- net OSC32_IN: now also Y2.2; no longer Q2.2
- net OSC32_OUT: now also Y2.1; no longer Q2.1
- net OSC_IN: now also Y1.2; no longer Q1.2
- net OSC_OUT: now also Y1.1; no longer Q1.1
Routing:
- net GND: track 8.01 -> 13.8 mm
- net N$5: track 6.28 -> 9.11 mm
- net PB2: track 6.31 -> 9.04 mm
- net VDD: track 253.2 -> 251.4 mm
- net N$25: track 39.2 -> 40.1 mm
- net +5VOUT: track 112.9 -> 113.4 mm
- net N$17: track 8.05 -> 8.56 mm
