File: hw/IRQF401RCT6v1.011.revB/IRQF401RCT6.sch (EAGLE design)
At the start: 105 parts, among them IC1 STM32F401RCT, IC2 LM1117IMPX-3.3, IC3 LM1117MPX-5.0, J2 RJ11, J3 RJ11, P1 FSM, Q1 8MHz, Q2 32.768kHz, Q3 BC846BSMD, Q4 BSS84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

Commit message: rev
New revision
Parts:
- renumbered Q1 to Y1, Q2 to Y2
